Commit message: add angle constraints for pendulum

File: quad/quad.urdf (robot description, URDF)
Before this commit: robot quadrotor_with_pendulum, 2 links, 1 joints
Links:
- added link ball, mass 0.5; visual sphere radius=0.06
- added link bar, mass 0.025; visual cylinder length=0.4 radius=0.015
- added link bar_tip, mass 0.025
Joints:
- added joint bar_ball: type fixed, parent bar, child ball, origin xyz=0.0 0.0 -0.4
- added joint x_revolution: type continuous, parent quadrotor, child bar_tip, axis 1.0 0.0 0.0
- added joint y_revolution: type continuous, parent bar_tip, child bar, axis 0.0 1.0 0.0
